Commit message: ⚡️ [ADD] : Add Gazebo Differential Drive Controller inc. Yaml and Launch files, and URDF Update

File: lenna_ws/src/lenna_description/urdf/lenna_description.urdf (robot description, URDF)
Before this commit: robot lenna_description, 6 links, 5 joints
Joints:
- removed joint base_joint
- added joint world_joint: type fixed, parent world, child base_link, origin xyz=0.0 0.0 0.02 rpy=0 0 0

Commit message: 🐛 [FIX] : Remove Fixed World Link, Making The Robot to Move in Gazebo

File: lenna_ws/src/lenna_description/urdf/lenna_description.urdf (robot description, URDF)
Before this commit: robot lenna_description, 6 links, 5 joints
Links:
- removed link world
Joints:
- removed joint world_joint
- joint left_wheel_joint: origin xyz=6.9033E-05 0.08975 0.014 rpy=-1.5708 0 0 -> xyz=6.9033E-05 0.08975 0.0150125 rpy=-1.5708 0 0
- joint right_wheel_joint: origin xyz=6.9033E-05 -0.08975 0.014 rpy=1.5708 0 0 -> xyz=6.9033E-05 -0.08975 0.0150125 rpy=1.5708 0 0
